File: board/board.kicad_pcb (KiCad board)
At the start: 2 copper layers, 21 x 13 mm, 1 part

Commit message: updated schemetic and layout
Parts:
- added C1: 100nF, Capacitor_SMD:C_0603_1608Metric, F.Cu at (143.9, 72.7)
- added C10: 100nF, Capacitor_SMD:C_0603_1608Metric, F.Cu at (155.4, 72.7)
- added C11: 100nF, Capacitor_SMD:C_0603_1608Metric, F.Cu at (149.4, 72.7)
- added C12: 100nF, Capacitor_SMD:C_0603_1608Metric, F.Cu at (141.8, 80.9)
- added C13: 2.2uF, Capacitor_SMD:C_0603_1608Metric, F.Cu at (154.4, 75.4)
- added C14: 2.2uF, Capacitor_SMD:C_0603_1608Metric, F.Cu at (156.9, 72.7)
- added C15: 22nF, Capacitor_SMD:C_0603_1608Metric, B.Cu at (154.4, 28.9)
- added C16: 100nF, Capacitor_SMD:C_0603_1608Metric, B.Cu at (144.6, 35.2)
- added C17: 100nF, Capacitor_SMD:C_0603_1608Metric, B.Cu at (142.2, 30.9)
- added C18: 6.8nF, Capacitor_SMD:C_0603_1608Metric, F.Cu at (154.4, 36.2)
- added C19: 100nF, Capacitor_SMD:C_0603_1608Metric, B.Cu at (146.4, 28.4)
- added C2: 12pF, Capacitor_SMD:C_0603_1608Metric, F.Cu at (150.8, 89.9)
- added C20: 6.8nF, Capacitor_SMD:C_0603_1608Metric, F.Cu at (154.4, 37.7)
- added C21: 100nF, Capacitor_SMD:C_0603_1608Metric, B.Cu at (144.9, 28.4)
- added C22: 10nF, Capacitor_SMD:C_0603_1608Metric, B.Cu at (154.4, 32.5)
- added C23: 100nF, Capacitor_SMD:C_0603_1608Metric, F.Cu at (152.0, 31.8)
- added C24: 10nF, Capacitor_SMD:C_0603_1608Metric, B.Cu at (142.2, 33.9)
- added C25: 4.7u, Capacitor_SMD:C_0603_1608Metric, B.Cu at (142.2, 32.4)
- added C26: 18pF, Capacitor_SMD:C_0603_1608Metric, F.Cu at (146.8, 43.4)
- added C27: 18pF, Capacitor_SMD:C_0603_1608Metric, F.Cu at (141.8, 38.0)
- added C3: 100nF, Capacitor_SMD:C_0603_1608Metric, F.Cu at (147.9, 72.7)
- added C4: 12pF, Capacitor_SMD:C_0603_1608Metric, F.Cu at (149.3, 89.9)
- added C5: 100nF, Capacitor_SMD:C_0603_1608Metric, F.Cu at (154.5, 61.7)
- added C6: 100nF, Capacitor_SMD:C_0603_1608Metric, F.Cu at (153.9, 72.7)
- added C7: 1nF, Capacitor_SMD:C_0603_1608Metric, F.Cu at (153.0, 85.6)
- added C8: 100nF, Capacitor_SMD:C_0603_1608Metric, F.Cu at (152.3, 89.9)
- added C9: 2.2uF, Capacitor_SMD:C_0603_1608Metric, F.Cu at (153.8, 89.9)
- added FB1: Ferrite_Bead_Small, Inductor_SMD:L_0805_2012Metric, F.Cu at (147.1, 61.0)
- added J1: UART, on_edge:on_edge_2x05_device, F.Cu at (140.0, 48.5)
- added J2: 008_USB, on_edge:on_edge_2x05_device, F.Cu at (140.0, 64.5)
- added J3: DebugEdge_02x05, on_edge:debug_edge_2x05_device, F.Cu at (140.0, 96.5)
- added J4: 019_100BASE-T_with_CT, on_edge:on_edge_2x05_host, F.Cu at (161.0, 32.5)
- added J5: ADC_2x3, on_edge:on_edge_2x05_host, F.Cu at (161.0, 48.5)
- added J7: SPI_2x3, on_edge:on_edge_2x05_host, F.Cu at (161.0, 96.5)
- added J8: I2C_2x2, on_edge:on_edge_2x05_host, F.Cu at (161.0, 80.5)
- added J9: UART_2x2, on_edge:on_edge_2x05_host, F.Cu at (161.0, 64.5)
- added R1: 27R, Resistor_SMD:R_0603_1608Metric, F.Cu at (152.4, 72.7)
- added R10: 10k, Resistor_SMD:R_0603_1608Metric, B.Cu at (154.0, 82.1)
- added R11: 10k, Resistor_SMD:R_0603_1608Metric, B.Cu at (154.0, 62.5)
- added R12: d.n.p, Resistor_SMD:R_0603_1608Metric, F.Cu at (150.5, 60.9)
- added R13: 10k, Resistor_SMD:R_0603_1608Metric, F.Cu at (155.3, 89.9)
- added R14: 1k, Resistor_SMD:R_0603_1608Metric, F.Cu at (149.3, 86.9)
- added R15: 200R, Resistor_SMD:R_0603_1608Metric, F.Cu at (153.7, 45.6)
- added R16: 1R, Resistor_SMD:R_0603_1608Metric, F.Cu at (153.7, 47.1)
- added R17: 49.9R, Resistor_SMD:R_0805_2012Metric, B.Cu at (154.2, 34.3)
- added R18: 3.3R, Resistor_SMD:R_0603_1608Metric, F.Cu at (151.4, 37.7)
- added R19: 3.3R, Resistor_SMD:R_0603_1608Metric, F.Cu at (151.4, 36.2)
- added R2: 27R, Resistor_SMD:R_0603_1608Metric, F.Cu at (150.9, 72.7)
- added R20: 3.3R, Resistor_SMD:R_0603_1608Metric, F.Cu at (152.0, 28.3)
- added R21: 3.3R, Resistor_SMD:R_0603_1608Metric, F.Cu at (152.0, 26.8)
- added R22: 12.4k, Resistor_SMD:R_0603_1608Metric, B.Cu at (143.4, 28.4)
- added R23: 1M, Resistor_SMD:R_0603_1608Metric, F.Cu at (144.8, 38.0)
- added R3: 10R, Resistor_SMD:R_0805_2012Metric, B.Cu at (154.2, 30.7)
- added R4: 49.9R, Resistor_SMD:R_0805_2012Metric, F.Cu at (154.9, 27.9)
- added R5: 49.9R, Resistor_SMD:R_0805_2012Metric, F.Cu at (152.2, 30.1)
- added R6: 49.9R, Resistor_SMD:R_0805_2012Metric, B.Cu at (154.2, 36.3)
- added R7: 2k, Resistor_SMD:R_0603_1608Metric, B.Cu at (154.0, 79.0)
- added R8: 2k, Resistor_SMD:R_0603_1608Metric, B.Cu at (154.0, 80.6)
- added R9: 10k, Resistor_SMD:R_0603_1608Metric, B.Cu at (154.3, 96.5)
- added U1: W25Q128JVS, Package_SO:SOIC-8_5.23x5.23mm_P1.27mm, F.Cu at (150.5, 66.5)
- added U2: RP2040, b018:RP2040-QFN-56, F.Cu at (149.0, 80.5)
- added U3: W5500, Package_QFP:LQFP-48_7x7mm_P0.5mm, F.Cu at (145.3, 32.1)
- added U4: 11AA02E48, Package_TO_SOT_SMD:SOT-23, F.Cu at (152.6, 93.4)
- added Y1: 12MhZ, Crystal:Crystal_SMD_Abracon_ABM8G-4Pin_3.2x2.5mm, F.Cu at (146.4, 89.0)
- added Y2: 25MHz, Crystal:Crystal_SMD_5032-2Pin_5.0x3.2mm, F.Cu at (143.3, 40.7)
- LOGO1: moved to B.Cu
- moved LOGO1 42.8 mm to (151.3, 56.2), turned to 180 degrees
Routing:
- net GND: track 0.00 -> 263.6 mm, vias 0 -> 25
- net +3V3: track 0.00 -> 194.2 mm, vias 0 -> 18
- net +5V: track 0.00 -> 90.0 mm, vias 0 -> 6
- net /controller/VDD: track 0.00 -> 61.2 mm, vias 0 -> 7
- net /rp2040/GPIO7: track 0.00 -> 58.0 mm, vias 0 -> 2
- net /rp2040/GPIO6: track 0.00 -> 56.3 mm, vias 0 -> 2
- net /rp2040/~{SPI0_CS}: track 0.00 -> 51.8 mm, vias 0 -> 2
- net /GPIO25: track 0.00 -> 51.6 mm, vias 0 -> 2
- net /rp2040/SPI0_RX: track 0.00 -> 51.4 mm, vias 0 -> 2
- net /rp2040/SPI0_TX: track 0.00 -> 50.8 mm, vias 0 -> 2
- net /rp2040/SPI0_SCK: track 0.00 -> 47.9 mm, vias 0 -> 2
- net /UART0_RX: track 0.00 -> 42.2 mm, vias 0 -> 2
- net /UART0_TX: track 0.00 -> 42.1 mm, vias 0 -> 2
- net /GPIO24: track 0.00 -> 41.9 mm, vias 0 -> 2
- net /ADC3: track 0.00 -> 38.6 mm, vias 0 -> 2
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Other:
- board size 21 x 13 mm -> 21 x 77 mm
- copper layers 2 -> 4
- board text added: "Debug"
- board text added: "osf.001"
- board text added: "osf.002"
- board text added: "osf.007"
- board text added: "osf.008 USB"
- board text added: "osf.010"
- board text added: "osf.010 UART"
- board text added: "osf.c001.v1.0"
