File: board/controller.kicad_sch (KiCad schematic)
At the start: 28 parts, among them U3 W5500, Y1 25MhZ

Commit message: added lcsc part numbers
Parts:
- C15: lcsc (none) -> C21122
- C16, C17, C19, C21, C23: DigiKey Part Number 1276-1012-1-ND -> (none); lcsc (none) -> C1525
- C18, C20: lcsc (none) -> C1631
- C22, C24: lcsc (none) -> C15195
- C25: lcsc (none) -> C23733
- C26, C27: DigiKey Part Number 1276-1089-1-ND -> (none); lcsc (none) -> C1549
- C30: lcsc (none) -> C1525
- R17, R4, R5, R6: lcsc (none) -> C17720
- R18, R19, R20, R21: lcsc (none) -> C22978
- R22: DigiKey Part Number 311-12.4KHRCT-ND -> (none); lcsc (none) -> C22865
- R23: DigiKey Part Number 311-1.0MGRCT-ND -> (none); lcsc (none) -> C26083
- R3: lcsc (none) -> C25077
- U3: DigiKey Part Number 1278-1021-ND -> (none); lcsc (none) -> C32843
- Y1: lcsc (none) -> C9006
Changed lines of the file:
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@@
       (effects (font (size 1.27 1.27)) hide)
     )
-    (property "DigiKey Part Number" "1276-1012-1-ND" (at 95.25 58.42 0)
+    (property "lcsc" "C1525" (at 95.25 58.42 0)
       (effects (font (size 1.27 1.27)) hide)
     )
@@
       (effects (font (size 1.27 1.27)) hide)
     )
+    (property "lcsc" "C17720" (at 96.52 116.84 0)
+      (effects (font (size 1.27 1.27)) hide)
+    )
     (pin "1")
     (pin "2")
@@
       (effects (font (size 1.27 1.27)) hide)
     )
+    (property "lcsc" "C23733" (at 179.07 109.22 0)
+      (effects (font (size 1.27 1.27)) hide)
+    )
     (pin "1")
     (pin "2")
@@
       (effects (font (size 1.27 1.27)) hide)
     )
+    (property "lcsc" "C1631" (at 74.93 87.63 0)
+      (effects (font (size 1.27 1.27)) hide)
+    )
     (pin "1")
     (pin "2")
@@
       (effects (font (size 1.27 1.27)) hide)
     )
+    (property "lcsc" "C17720" (at 88.9 116.84 0)
+      (effects (font (size 1.27 1.27)) hide)
+    )
     (pin "1")
     (pin "2")
@@
       (effects (font (size 1.27 1.27)) hide)
     )
+    (property "lcsc" "C22978" (at 116.84 95.25 0)
+      (effects (font (size 1.27 1.27)) hide)
+    )
     (pin "1")
     (pin "2")
@@
       (effects (font (size 1.27 1.27)) hide)
     )
+    (property "lcsc" "" (at 104.775 121.92 0)
+      (effects (font (size 1.27 1.27)) hide)
+    )
     (pin "1")
     (pin "2")
@@
       (effects (font (size 1.27 1.27)) hide)
     )
+    (property "lcsc" "C22978" (at 105.41 90.17 0)
+      (effects (font (size 1.27 1.27)) hide)
+    )
     (pin "1")
     (pin "2")
@@
       (effects (font (size 1.27 1.27)) hide)
     )
-    (property "DigiKey Part Number" "1276-1012-1-ND" (at 80.01 58.42 0)
+    (property "lcsc" "C1525" (at 80.01 58.42 0)
       (effects (font (size 1.27 1.27)) hide)
     )
@@
       (effects (font (size 1.27 1.27)) hide)
     )
-    (property "DigiKey Part Number" "311-1.0MGRCT-ND" (at 176.53 87.63 0)
+    (property "lcsc" "C26083" (at 176.53 87.63 0)
       (effects (font (size 1.27 1.27)) hide)
     )
@@
       (effects (font (size 1.27 1.27)) (justify left) hide)
     )
-    (property "DigiKey Part Number" "1278-1021-ND" (at 133.35 34.29 0)
-      (effects (font (size 1.27 1.27)) (justify left) hide)
+    (property "lcsc" "C32843" (at 143.51 86.36 0)
+      (effects (font (size 1.27 1.27)) hide)
     )
     (pin "1")
@@
       (effects (font (size 1.27 1.27)) hide)
     )
+    (property "lcsc" "C1525" (at 109.855 125.73 0)
+      (effects (font (size 1.27 1.27)) hide)
+    )
     (pin "1")
     (pin "2")
@@
       (effects (font (size 1.27 1.27)) hide)
     )
+    (property "lcsc" "C22978" (at 110.49 87.63 0)
+      (effects (font (size 1.27 1.27)) hide)
+    )
     (pin "1")
     (pin "2")
@@
       (effects (font (size 1.27 1.27)) hide)
     )
-    (property "DigiKey Part Number" "311-12.4KHRCT-ND " (at 168.91 109.22 0)
+    (property "lcsc" "C22865" (at 168.91 109.22 0)
       (effects (font (size 1.27 1.27)) hide)
     )
@@
       (effects (font (size 1.27 1.27)) hide)
     )
-    (property "DigiKey Part Number" "1276-1012-1-ND" (at 64.77 58.42 0)
+    (property "lcsc" "C1525" (at 64.77 58.42 0)
       (effects (font (size 1.27 1.27)) hide)
     )
@@
       (effects (font (size 1.27 1.27)) hide)
     )
+    (property "lcsc" "C15195" (at 92.71 125.73 0)
+      (effects (font (size 1.27 1.27)) hide)
+    )
     (pin "1")
     (pin "2")
@@
       (effects (font (size 1.27 1.27)) hide)
     )
+    (property "lcsc" "C25077" (at 55.88 118.11 0)
+      (effects (font (size 1.27 1.27)) hide)
+    )
     (pin "1")
     (pin "2")
@@
       (effects (font (size 1.27 1.27)) hide)
     )
-    (property "DigiKey Part Number" "1276-1012-1-ND" (at 87.63 58.42 0)
+    (property "lcsc" "C1525" (at 87.63 58.42 0)
       (effects (font (size 1.27 1.27)) hide)
     )
@@
       (effects (font (size 1.27 1.27)) hide)
     )
+    (property "lcsc" "C17720" (at 62.23 81.28 0)
+      (effects (font (size 1.27 1.27)) hide)
+    )
     (pin "1")
     (pin "2")
@@
       (effects (font (size 1.27 1.27)) hide)
     )
+    (property "lcsc" "C21122" (at 55.88 125.73 0)
+      (effects (font (size 1.27 1.27)) hide)
+    )
     (pin "1")
     (pin "2")
@@
       (effects (font (size 1.27 1.27)) hide)
     )
+    (property "lcsc" "C22978" (at 123.19 92.71 0)
+      (effects (font (size 1.27 1.27)) hide)
+    )
     (pin "1")
     (pin "2")
@@
     )
     (property "Datasheet" "~" (at 163.83 87.63 0)
+      (effects (font (size 1.27 1.27)) hide)
+    )
+    (property "lcsc" "C9006" (at 163.83 87.63 0)
       (effects (font (size 1.27 1.27)) hide)
     )
@@
       (effects (font (size 1.27 1.27)) hide)
     )
-    (property "DigiKey Part Number" "1276-1089-1-ND" (at 189.23 109.22 0)
+    (property "lcsc" "C1549" (at 189.23 109.22 0)
       (effects (font (size 1.27 1.27)) hide)
     )
@@
       (effects (font (size 1.27 1.27)) hide)
     )
-    (property "DigiKey Part Number" "1276-1089-1-ND" (at 199.39 109.22 0)
+    (property "lcsc" "C1549" (at 199.39 109.22 0)
       (effects (font (size 1.27 1.27)) hide)
     )
@@
       (effects (font (size 1.27 1.27)) hide)
     )
+    (property "lcsc" "C1631" (at 81.28 90.17 0)
+      (effects (font (size 1.27 1.27)) hide)
+    )
     (pin "1")
     (pin "2")
@@
       (effects (font (size 1.27 1.27)) hide)
     )
+    (property "lcsc" "C15195" (at 113.03 64.77 0)
+      (effects (font (size 1.27 1.27)) hide)
+    )
     (pin "1")
     (pin "2")
@@
       (effects (font (size 1.27 1.27)) hide)
     )
-    (property "DigiKey Part Number" "1276-1012-1-ND" (at 72.39 58.42 0)
+    (property "lcsc" "C1525" (at 72.39 58.42 0)
       (effects (font (size 1.27 1.27)) hide)
     )
@@
       (effects (font (size 1.27 1.27)) hide)
     )
+    (property "lcsc" "C17720" (at 69.85 81.28 0)
+      (effects (font (size 1.27 1.27)) hide)
+    )
